File: blueprint/pcb/1.5.1/Goalfinder.kicad_sch (KiCad schematic)
At the start: 42 parts, among them J1 USB in, J1-Board1 USB_B_Micro_Breakout, J2 USB-ESP, J3 GAIN, J4 LED Strip, J4e1 Conn_01x02_Pin, J5 SW240 - Vcc/D0/GND, J5e1 Conn_01x03_Socket, J6 VL53L0X-ToF Vcc/SDA/SCL/GND, J7 Conn_01x08_Pin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

Commit message: Cleared PCB
Parts:
- J2: footprint Connector_PinHeader_2.54mm:PinHeader_1x04_P2.54mm_Vertical -> Connector_JST:JST_XH_B4B-XH-A_1x04_P2.50mm_Vertical
- J3: footprint Connector_PinHeader_2.54mm:PinHeader_2x05_P2.54mm_Vertical -> (none)
- J5: footprint Connector_PinSocket_2.54mm:PinSocket_1x03_P2.54mm_Vertical -> Connector_JST:JST_XH_B3B-XH-A_1x03_P2.50mm_Vertical
- J7: footprint (none) -> Connector_PinSocket_2.54mm:PinSocket_1x08_P2.54mm_Vertical
- U5: footprint Sensor_Motion:InvenSense_QFN-24_4x4mm_P0.5mm -> (none)
Changed lines of the file:
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@@
 			)
 		)
-		(property "Footprint" ""
+		(property "Footprint" "Connector_PinSocket_2.54mm:PinSocket_1x08_P2.54mm_Vertical"
 			(at 187.96 121.92 0)
 			(effects
@@
 			)
 		)
-		(property "Footprint" "Connector_PinHeader_2.54mm:PinHeader_1x04_P2.54mm_Vertical"
+		(property "Footprint" "Connector_JST:JST_XH_B4B-XH-A_1x04_P2.50mm_Vertical"
 			(at 250.19 22.86 0)
 			(effects
@@
 			)
 		)
-		(property "Footprint" "Connector_PinSocket_2.54mm:PinSocket_1x03_P2.54mm_Vertical"
+		(property "Footprint" "Connector_JST:JST_XH_B3B-XH-A_1x03_P2.50mm_Vertical"
 			(at 54.61 76.2 0)
 			(effects
@@
 			)
 		)
-		(property "Footprint" "Connector_PinHeader_2.54mm:PinHeader_2x05_P2.54mm_Vertical"
+		(property "Footprint" ""
 			(at 114.3 67.056 0)
 			(effects
@@
 			)
 		)
-		(property "Footprint" "Sensor_Motion:InvenSense_QFN-24_4x4mm_P0.5mm"
+		(property "Footprint" ""
 			(at 139.7 160.02 0)
 			(effects
